File: hardware/hardware-v3/thermostat.sch (EAGLE design)
At the start: 38 parts

Commit message: New Layout
Parts:
- removed C3: 100n, rcl:C-EUC0805
- removed CADDBUF: 100n, eagle-ltspice:CC0402
- removed R10, R12, R13, R16: 1k, rcl:R-EU_R0603
- removed R11, R3, R4, R5, R6, R7, R8: 47, resistor:R-EU_R0402
- removed R17, R18, R9: 10k, rcl:R-EU_R0603
- removed U$3: MCP4141-103, microchip:MCP4141-103
- added C4, C_CAP2: 100n, eagle-ltspice:CC0603
- added RA, RA1, RA2, RA3, RA4, RA5, RA6, RA7: 47, rcl:R-EU_R0603
- added RS1, RS2, RS3: 1k, rcl:R-EU_R0603
- added RT1, RT2, RT3: 10k, rcl:R-EU_R0603
- added S1: MOMENTARY-SWITCH-SPST-SMD-4.6X2.8MM, SparkFun-Switches:MOMENTARY-SWITCH-SPST-SMD-4.6X2.8MM
- added X1: USB-1X-2S-PLUG-A-SMD, _con-usb:USB-1X-2S-PLUG-A-SMD
- added X2: 332-02, con-garry:332-02
- C2: device rcl:C-EUC0805 -> eagle-ltspice:CC0603
- CBUF: device eagle-ltspice:CC0402 -> eagle-ltspice:CC0603
- R2: value 47 -> 1k; device resistor:R-EU_R0402 -> rcl:R-EU_R0603
- U$1: value MICRO-USB -> MCP4151; device microusb:MICRO-USB -> microchip:MCP4151
- renumbered R14 to RMCLR
Connections:
- removed net N$3: R16.1, U$3.P0B
- new net 3V3G: C2.1, R1.2, RT1.2, RT2.2, RT3.2, T1.E, T2.E, T3.E, U$1.P0B, U$1.VDD, X2-2.S
- new net N$30: S1.2, U$2.RB0/PGD1/AN0
- net +3V3: now also CBUF.1, C_CAP2.2, X2-1.S; no longer C3.2, CADDBUF.2, CBUF.2, R1.2, R16.2, R17.2, R18.2, R9.2, T1.E, T2.E, T3.E, U$3.VDD
- net A: now also RA.1; no longer R8.2
- net B: now also RA6.1; no longer R7.2
- net C: now also RA5.1; no longer R6.2
- net CS: now also U$1.NCS, U$2.RG3; no longer U$2.RC12, U$3.~CS
- net D: now also RA4.1; no longer R5.2
- net DP: now also RA7.1; no longer R11.2
- net E: now also RA3.1; no longer R4.2
- net F: now also RA2.1; no longer R3.2
- net G: now also RA1.1; no longer R2.2
- net GND: now also C4.2, CBUF.2, C_CAP2.1, S1.1, U$1.P0A, U$1.VSS, X1.4, X1.S1, X1.S2; no longer C3.1, CADDBUF.1, CBUF.1, U$1.GND, U$3.VSS
- net IN1: now also NTC.1, R1.1, U$2.RB14/AN14; no longer U$2.RB1/PGC1/AN1, U$3.P0W
- net IN2: now also U$1.P0W, U$2.RB15/AN15; no longer NTC.1, R1.1, U$2.RB0/PGD1/AN0
- net MCLR: now also C4.1; no longer C2.1
- net N$12: now also RS3.2, RT3.1; no longer R10.2, R18.1
- net N$14: now also RS2.2, RT2.1; no longer R12.2, R9.1
- net N$16: no longer DIS1.CA
- net N$17: no longer DIS2.CA
- net N$18: no longer DIS3.CA
- net N$5: now also RS1.2, RT1.1; no longer R13.2, R17.1
- net N$6: now also X1.1; no longer U$1.VCC
- net S1: now also RS1.1, U$2.RC13; no longer R13.1, U$2.RB15/AN15
- net S2: now also RS2.1, U$2.RC15; no longer R12.1, U$2.RB14/AN14
- net S3: now also RS3.1, U$2.RC12; no longer R10.1, U$2.RB10/AN10
- net SCK: now also U$1.SCK; no longer U$3.SCK
- net SDI: now also R2.1; no longer U$3.SDI
- net SDO: now also R2.2, U$1.SDI_SDO; no longer U$3.SDO
- net _A: now also RA.2, U$2.RE2; no longer R8.1, U$2.RC15
- net _B: now also RA6.2; no longer R7.1
- net _C: now also RA5.2; no longer R6.1
- net _D: now also RA4.2; no longer R5.1
- net _DP: now also RA7.2, U$2.RB1/PGC1/AN1; no longer R11.1, U$2.RE2
- net _E: now also RA3.2; no longer R4.1
- net _F: now also RA2.2; no longer R3.1
- net _G: now also RA1.2; no longer R2.1
Other:
- note removed: "NEED TO CHECK SIZES OF RESISTORS AND CAPACITORS"
- moved on the sheet: C2, CBUF, D2, NTC, R1, R2, T1, T2, T3
